File: pcb/tartan.kicad_pcb (KiCad board)
At the start: 2 copper layers, 285 x 117 mm, 171 parts, among them J1 AVR_ISP_6, J2 USB_OTG, SW1 SW_Push, SW10 SW_Push, SW11 SW_Push, SW12 SW_Push, SW13 SW_Push, SW14 SW_Push, SW15 SW_Push, SW16 SW_Push, SW17 SW_Push, SW18 SW_Push, SW19 SW_Push, SW2 SW_Push, SW20 SW_Push, SW21 SW_Push, SW22 SW_Push, SW23 SW_Push, SW24 SW_Push, SW25 SW_Push, SW26 SW_Push, SW27 SW_Push, SW28 SW_Push, SW29 SW_Push, SW3 SW_Push, SW30 SW_Push, SW31 SW_Push, SW32 SW_Push, SW33 SW_Push, SW34 SW_Push, SW35 SW_Push, SW36 SW_Push, SW37 SW_Push, SW38 SW_Push, SW39 SW_Push, SW4 SW_Push, SW40 SW_Push, SW41 SW_Push, SW42 SW_Push, SW43 SW_Push, SW44 SW_Push, SW45 SW_Push, SW46 SW_Push, SW47 SW_Push, SW48 SW_Push, SW49 SW_Push, SW5 SW_Push, SW50 SW_Push, SW51 SW_Push, SW52 SW_Push, SW53 SW_Push, SW54 SW_Push, SW55 SW_Push, SW56 SW_Push, SW57 SW_Push, SW58 SW_Push, SW59 SW_Push, SW6 SW_Push, SW60 SW_Push, SW61 SW_Push, SW62 SW_Push, SW63 SW_Push, SW64 SW_Push, SW65 SW_Push, SW66 SW_Push, SW67 SW_Push, SW68 SW_Push, SW69 SW_Push, SW7 SW_Push, SW70 RESET, SW71 BOOT, SW8 SW_Push, SW9 SW_Push, U1 ATMEGA328-PU, Y1 16MHz

Commit message: Update tartan.kicad_pcb
swapped out mini usb connector for micro usb
Parts:
- J2: footprint dm9_conn:USB_MINIB_Akizuki_MUSB-5BF01AS -> Connector_USB:USB_Micro-B_Amphenol_10103594-0001LF_Horizontal
- moved J2 6.77 mm to (266.8, 32.9)
Routing:
- net GND: track 13.4 -> 18.4 mm
- net Net-(F1-Pad1): track 3.56 -> 8.11 mm
- net Net-(D66-Pad1): track 18.4 -> 20.9 mm

Commit message: Added gerber files
Parts:
- removed G***: LOGO, tartan:band
-  : renamed from G***; value LOGO -> (none); footprint tartan:logo1 -> Battery:yay
